File: hardware/neogeo-diag-aes-prog.kicad_pcb (KiCad board)
At the start: 2 copper layers, 174 x 134 mm, 19 parts, among them J1 neogeo-aes-prog-a-side-edge, J2 neogeo-aes-prog-a-side-edge, J3 neogeo-aes-prog-b-side-edge, J4 neogeo-aes-prog-b-side-edge, U1 AS6C8016, U2 74LS08, U3 74LS11, U4 74LS04

Commit message: Fix silkscreen typo 68KCLB -> 68KCLKB
Other:
- board text added: "68KCLKB"
- board text removed: "68KCLB"

Commit message: Add logo
Parts:
- added G***: LOGO, neogeo-diag:neogeo-diag-aes-prog-logo, F.Cu at (203.2, 39.9)
- added G***: LOGO, neogeo-diag:neogeo-diag-aes-prog-logo, B.Cu at (202.9, 39.9)
- moved REF** 1.80 mm to (67.8, 40.4)
- moved REF** 1.78 mm to (67.8, 40.6)
Other:
- board text added: "REV ${REV}"
- board text removed: "NEOGEO DIAG AES PROG ${REV}"
